Commit message: next step done

File: src/armbot_description/urdf/armbot.urdf.xacro (robot description, xacro)
@@ -1,177 +1,228 @@
 <?xml version="1.0"?>
-<robot xmlns:xacro="http://www.ros.org/wiki/xacro">
-  <link name="base_link">
-	  <visual>
-        <geometry>
-          <mesh filename="file:///$(find smart_arm)/description/meshes/base_cylinder.stl" scale ="0.0001 0.0001 0.0001"/>
-        </geometry>
-        <origin xyz="0 0 0.01"/>
-        <material name="black">
-           <color rgba="0 0 0 1 "/>
-        </material>
-    </visual>
-	  <collision>
-        <geometry>
-          <mesh filename="file:///$(find smart_arm)/description/meshes/base_cylinder.stl" scale ="0.0001 0.0001 0.0001"/>
-        </geometry>
-        <origin xyz="0 0 0.01"/>
-    </collision>
-  </link>
-  <link name="platform">
-      <visual>
-          <geometry>
-              <mesh filename="file:///$(find smart_arm)/description/meshes/top_plate.stl" scale ="0.001 0.001 0.001"/>
-          </geometry>
-          <origin xyz="0 0 0"/>
-          <material name="black"/>
-      </visual>
-      <collision>
-        <geometry>
-          <mesh filename="file:///$(find smart_arm)/description/meshes/top_plate.stl" scale ="0.001 0.001 0.001"/>
-        </geometry>
-        <origin xyz="0 0 0"/>
-      </collision>
-  </link>
-  <link name="lower_arm">
-      <visual>
-          <geometry>
-              <mesh filename="file:///$(find smart_arm)/description/meshes/lower_arm.stl" scale ="0.001 0.001 0.001"/>
-          </geometry>
-          <origin xyz="0 0 0"/>
-          <material name="black"/>
-      </visual>
-      <collision>
-          <geometry>
-            <mesh filename="file:///$(find smart_arm)/description/meshes/lower_arm.stl" scale ="0.001 0.001 0.001"/>
-          </geometry>
-          <origin xyz="0 0 0"/>
-      </collision>
-  </link>
-  <link name="top_arm">
-      <visual>
-        <geometry>
-          <mesh filename="file:///$(find smart_arm)/description/meshes/top_arm.stl" scale ="0.001 0.001 0.001"/>
-        </geometry>
-        <origin rpy="0 1.59 0" xyz="0 0 0"/>
-        <material name="black"/>
-      </visual>
-      <collision>
-          <geometry>
-              <mesh filename="file:///$(find smart_arm)/description/meshes/top_arm.stl" scale ="0.001 0.001 0.001"/>
-          </geometry>
-          <origin rpy="0 1.59 0" xyz="0 0 0"/>
-      </collision>
-  </link>
-  <link name="wrist">
-      <visual>
-        <geometry>
-          <mesh filename="file:///$(find smart_arm)/description/meshes/wrist.stl" scale ="0.001 0.001 0.001"/>
-        </geometry>
-        <origin rpy="0 0 0" xyz="0 0 0"/>
-        <material name="black"/>
-      </visual>
-      <collision>
-        <geometry>
-          <mesh filename="file:///$(find smart_arm)/description/meshes/wrist.stl" scale ="0.001 0.001 0.001"/>
-        </geometry>
-        <origin rpy="0 0 0" xyz="0 0 0"/>
-      </collision>
-  </link>
-  <link name="clawbase">
-      <visual>
-          <geometry>
-            <mesh filename="file:///$(find smart_arm)/description/meshes/clawbase.stl" scale ="0.001 0.001 0.001"/>
-          </geometry>
-          <origin rpy="0 3.18 0" xyz="0 0 0"/>
-          <material name="white">
-            <color rgba="1 1 1 1"/>
-          </material>
-      </visual>
-      <collision>
-          <geometry>
-            <mesh filename="file:///$(find smart_arm)/description/meshes/clawbase.stl" scale ="0.001 0.001 0.001"/>
-          </geometry>
-          <origin rpy="0 3.18 0" xyz="0 0 0"/>
-      </collision>
-  </link>
-  <link name="clawr">
-      <visual>
-          <geometry>
-            <mesh filename="file:///$(find smart_arm)/description/meshes/clawr.stl" scale ="0.001 0.001 0.001"/>
-          </geometry>
-          <origin rpy="0 0 0" xyz="0 0 0"/>
-          <material name="white"/>
-      </visual>
-      <collision>
-          <geometry>
-            <mesh filename="file:///$(find smart_arm)/description/meshes/clawr.stl" scale ="0.001 0.001 0.001"/>
-          </geometry>
-          <origin rpy="0 0 0" xyz="0 0 0"/>
-      </collision>
-  </link>
-  <link name="clawl">
-	<visual>
-         <geometry>
-          <mesh filename="file:///$(find smart_arm)/description/meshes/clawl.stl" scale ="0.001 0.001 0.001"/>
-         </geometry>
-         <material name="white"/>
-         <origin rpy="0 0 0" xyz="0 0 0"/>
-      </visual>
-	<collision>
-         <geometry>
-          <mesh filename="file:///$(find smart_arm)/description/meshes/clawl.stl" scale ="0.001 0.001 0.001"/>
-         </geometry>
-         <origin rpy="0 0 0" xyz="0 0 0"/>
-        </collision>
-  </link>
-  <joint name="joint1" type="revolute">
-    <axis xyz="0 0 1" />
-    <limit effort="1000.0" lower="1.56" upper="4.68" velocity="1.0" />
-    <parent link="base_link"/>
-    <child link="platform"/>
-    <origin rpy="0 0 1.5" xyz="0 0 0.48"/>
-  </joint>
-  <joint name="joint2" type="revolute">
-    <axis xyz="1 0 0" />
-    <limit effort="1000.0" lower="0.0" upper="3.12" velocity="1.0" />
-    <parent link="platform"/>
-    <child link="lower_arm"/>
-    <origin xyz="0 0.19 0.28"/>
-  </joint>
-  <joint name="joint3" type="revolute">
-    <axis xyz="1 0 0" />
-    <limit effort="1000.0" lower="-1.7" upper="1.7" velocity="1.0" />
-    <parent link="lower_arm"/>
-    <child link="top_arm"/>
-    <origin xyz="-0.25 1.0 0"/>
-  </joint>
-  <joint name="joint4" type="revolute">
-    <axis xyz="1 0 0" />
-    <limit effort="1000.0" lower="-1.7" upper="1.7" velocity="1.0" />
-    <parent link="top_arm"/>
-    <child link="wrist"/>
-    <origin xyz="0.11 1.25 0"/>
-  </joint>
-  <joint name="joint5" type="revolute">
-    <axis xyz="0 1 0" />
-    <limit effort="1000.0" lower="-3.17" upper="0.0" velocity="1.0" />
-    <parent link="wrist"/>
-    <child link="clawbase"/>
-    <origin xyz="0 0.63 0"/>
-  </joint>
-  <joint name="joint6" type="revolute">
-    <axis xyz="0 0 1" />
-    <limit effort="1000.0" lower="-0.5" upper="0.0" velocity="1.0" />
-    <parent link="clawbase"/>
-    <child link="clawr"/>
-    <origin rpy="0 0 -0.31" xyz="0.11 0.34 0"/>
-  </joint>
-  <joint name="joint7" type="revolute">
-    <axis xyz="0 0 1" />
-    <limit effort="1000.0" lower="0" upper="-0.5" velocity="1.0" />
-    <parent link="clawbase"/>
-    <child link="clawl"/>
-    <origin rpy="0 0 0.22" xyz="-0.16 0.30 0"/>
-    <mimic joint="joint6" multiplier="-1" offset="0" />
-  </joint>
+<robot xmlns:xacro="http://www.ros.org/wiki/xacro" name="armbot">
+    <!-- Include Gazebo Parameters -->
+    <xacro:include filename="$(find armbot_description)/urdf/armbot_gazebo.xacro" />
+    <!-- Include ros2_control Plugins -->
+    <xacro:include filename="$(find armbot_description)/urdf/armbot_ros2_control.xacro" />
+    <!-- Useful XACRO Variables (Properties) -->
+    <xacro:property name="PI" value="3.14159265359" />
+    <xacro:property name="effort" value="1000.0" />
+    <xacro:property name="velocity" value="1.0" />
+    <!-- Useful Macros -->
+    <xacro:macro name="default_inertial" params="mass">
+        <inertial>
+            <origin xyz="0 0 0" rpy="0 0 0"/>
+            <mass value="${mass}" />
+            <inertia ixx="1.0" ixy="0.0" ixz="0.0"
+                     iyy="1.0" iyz="0.0"
+                     izz="1.0" />
+        </inertial>
+    </xacro:macro>
+    <xacro:macro name="default_transmission" params="number">
+        <transmission name="transmission_${number}">
+            <plugin>transmission_interface/SimpleTransmission</plugin>
+            <actuator name="motor_${number}" role="actuator1"/>
+            <joint name="joint_${number}"    role="joint1">
+                <mechanical_reduction>1.0</mechanical_reduction>
+            </joint>
+        </transmission>
+    </xacro:macro>
+    <!-- Links -->
+    <link name="world"/>
+    <link name="base_link">
+        <xacro:default_inertial mass="1.0"/>
+        <visual>
+            <origin rpy="0 0 0" xyz="0 0 0.01"/>
+            <geometry>
+                <mesh filename="package://armbot_description/meshes/base_cylinder.stl" scale="0.0001 0.0001 0.0001"/>
+            </geometry>
+            <material name="black">
+                <color rgba="0 0 0 1"/>
+            </material>
+        </visual>
+        <collision>
+            <origin rpy="0 0 0" xyz="0 0 0.01"/>
+            <geometry>
+                <mesh filename="package://armbot_description/meshes/base_cylinder.stl" scale="0.0001 0.0001 0.0001"/>
+            </geometry>
+        </collision>
+    </link>
+    <link name="platform">
+        <xacro:default_inertial mass="0.5"/>
+        <visual>
+            <origin rpy="0 0 0" xyz="0 0 0"/>
+            <geometry>
+                <mesh filename="package://armbot_description/meshes/top_plate.stl" scale="0.001 0.001 0.001"/>
+            </geometry>
+            <material name="black"/>
+        </visual>
+        <collision>
+            <origin rpy="0 0 0" xyz="0 0 0"/>
+            <geometry>
+                <mesh filename="package://armbot_description/meshes/top_plate.stl" scale="0.001 0.001 0.001"/>
+            </geometry>
+        </collision>
+    </link>
+    <link name="lower_arm">
+        <xacro:default_inertial mass="0.5"/>
+        <visual>
+            <origin rpy="0 0 0" xyz="0 0 0"/>
+            <geometry>
+                <mesh filename="package://armbot_description/meshes/lower_arm.stl" scale="0.001 0.001 0.001"/>
+            </geometry>
+            <material name="black"/>
+        </visual>
+        <collision>
+            <origin rpy="0 0 0" xyz="0 0 0"/>
+            <geometry>
+                <mesh filename="package://armbot_description/meshes/lower_arm.stl" scale="0.001 0.001 0.001"/>
+            </geometry>
+        </collision>
+    </link>
+    <link name="top_arm">
+        <xacro:default_inertial mass="0.5"/>
+        <visual>
+            <origin rpy="0 1.59 0" xyz="0 0 0"/>
+            <geometry>
+                <mesh filename="package://armbot_description/meshes/top_arm.stl" scale="0.001 0.001 0.001"/>
+            </geometry>
+            <material name="black"/>
+        </visual>
+        <collision>
+            <origin rpy="0 1.59 0" xyz="0 0 0"/>
+            <geometry>
+                <mesh filename="package://armbot_description/meshes/top_arm.stl" scale="0.001 0.001 0.001"/>
+            </geometry>
+        </collision>
+    </link>
+    <link name="wrist">
+        <xacro:default_inertial mass="0.5"/>
+        <visual>
+            <origin rpy="0 0 0" xyz="0 0 0"/>
+            <geometry>
+                <mesh filename="package://armbot_description/meshes/wrist.stl" scale="0.001 0.001 0.001"/>
+            </geometry>
+            <material name="black"/>
+        </visual>
+        <collision>
+            <origin rpy="0 0 0" xyz="0 0 0"/>
+            <geometry>
+                <mesh filename="package://armbot_description/meshes/wrist.stl" scale="0.001 0.001 0.001"/>
+            </geometry>
+        </collision>
+    </link>
+    <link name="clawbase">
+        <xacro:default_inertial mass="0.2"/>
+        <visual>
+            <origin rpy="0 3.18 0" xyz="0 0 0"/>
+            <geometry>
+                <mesh filename="package://armbot_description/meshes/clawbase.stl" scale="0.001 0.001 0.001"/>
+            </geometry>
+            <material name="white">
+                <color rgba="1 1 1 1"/>
+            </material>
+        </visual>
+        <collision>
+            <origin rpy="0 3.18 0" xyz="0 0 0"/>
+            <geometry>
+                <mesh filename="package://armbot_description/meshes/clawbase.stl" scale="0.001 0.001 0.001"/>
+            </geometry>
+        </collision>
+    </link>
+    <link name="clawr">
+        <xacro:default_inertial mass="0.1"/>
+        <visual>
+            <origin rpy="0 0 0" xyz="0 0 0"/>
+            <geometry>
+                <mesh filename="package://armbot_description/meshes/clawr.stl" scale="0.001 0.001 0.001"/>
+            </geometry>
+            <material name="white"/>
+        </visual>
+        <collision>
+            <origin rpy="0 0 0" xyz="0 0 0"/>
+            <geometry>
+                <mesh filename="package://armbot_description/meshes/clawr.stl" scale="0.001 0.001 0.001"/>
+            </geometry>
+        </collision>
+    </link>
+    <link name="clawl">
+        <xacro:default_inertial mass="0.1"/>
+        <visual>
+            <origin rpy="0 0 0" xyz="0 0 0"/>
+            <geometry>
+                <mesh filename="package://armbot_description/meshes/clawl.stl" scale="0.001 0.001 0.001"/>
+            </geometry>
+            <material name="white"/>
+        </visual>
+        <collision>
+            <origin rpy="0 0 0" xyz="0 0 0"/>
+            <geometry>
+                <mesh filename="package://armbot_description/meshes/clawl.stl" scale="0.001 0.001 0.001"/>
+            </geometry>
+        </collision>
+    </link>
+    <!-- Joints -->
+    <joint name="virtual_joint" type="fixed">
+        <parent link="world"/>
+        <child link="base_link"/>
+        <origin xyz="0 0 0" rpy="0 0 0"/>
+    </joint>
+    <joint name="joint_1" type="revolute">
+        <axis xyz="0 0 1" />
+        <limit effort="${effort}" lower="1.56" upper="4.68" velocity="${velocity}" />
+        <parent link="base_link"/>
+        <child link="platform"/>
+        <origin rpy="0 0 1.5" xyz="0 0 0.48"/>
+    </joint>
+    <joint name="joint_2" type="revolute">
+        <axis xyz="1 0 0" />
+        <limit effort="${effort}" lower="0.0" upper="3.12" velocity="${velocity}" />
+        <parent link="platform"/>
+        <child link="lower_arm"/>
+        <origin xyz="0 0.19 0.28"/>
+    </joint>
+    <joint name="joint_3" type="revolute">
+        <axis xyz="1 0 0" />
+        <limit effort="${effort}" lower="-1.7" upper="1.7" velocity="${velocity}" />
+        <parent link="lower_arm"/>
+        <child link="top_arm"/>
+        <origin xyz="-0.25 1.0 0"/>
+    </joint>
+    <joint name="joint_4" type="revolute">
+        <axis xyz="1 0 0" />
+        <limit effort="${effort}" lower="-1.7" upper="1.7" velocity="${velocity}" />
+        <parent link="top_arm"/>
+        <child link="wrist"/>
+        <origin xyz="0.11 1.25 0"/>
+    </joint>
+    <joint name="joint_5" type="revolute">
+        <axis xyz="0 1 0" />
+        <limit effort="${effort}" lower="-3.17" upper="0.0" velocity="${velocity}" />
+        <parent link="wrist"/>
+        <child link="clawbase"/>
+        <origin xyz="0 0.63 0"/>
+    </joint>
+    <joint name="joint_6" type="revolute">
+        <axis xyz="0 0 1" />
+        <limit effort="${effort}" lower="-0.5" upper="0.0" velocity="${velocity}" />
+        <parent link="clawbase"/>
+        <child link="clawr"/>
+        <origin rpy="0 0 -0.31" xyz="0.11 0.34 0"/>
+    </joint>
+    <joint name="joint_7" type="revolute">
+        <axis xyz="0 0 1" />
+        <limit effort="${effort}" lower="0" upper="-0.5" velocity="${velocity}" />
+        <parent link="clawbase"/>
+        <child link="clawl"/>
+        <origin rpy="0 0 0.22" xyz="-0.16 0.30 0"/>
+        <mimic joint="joint6" multiplier="-1" offset="0" />
+    </joint>
+    <!-- Transmissions -->
+    <xacro:default_transmission number="1" />
+    <xacro:default_transmission number="2" />
+    <xacro:default_transmission number="3" />
+    <xacro:default_transmission number="4" />
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