Commit message: next step for robotics arm control

File: src/armbot_description/urdf/armbot.urdf.xacro (robot description, xacro)
@@ -1,4 +1,6 @@
 <?xml version="1.0"?>
 <robot xmlns:xacro="http://www.ros.org/wiki/xacro" name="armbot">
+    <!-- Load Simulated or Real Hardware Interfaces -->
+    <xacro:arg name="is_sim" default="true"/>
     <!-- Include Gazebo Parameters -->
     <xacro:include filename="$(find armbot_description)/urdf/armbot_gazebo.xacro" />
@@ -12,9 +14,9 @@
     <xacro:macro name="default_inertial" params="mass">
         <inertial>
-            <origin xyz="0 0 0" rpy="0 0 0"/>
+            <origin xyz="0 0 0" rpy="0 0 0" />
             <mass value="${mass}" />
             <inertia ixx="1.0" ixy="0.0" ixz="0.0"
-                     iyy="1.0" iyz="0.0"
-                     izz="1.0" />
+                iyy="1.0" iyz="0.0"
+                izz="1.0" />
         </inertial>
     </xacro:macro>
@@ -22,6 +24,6 @@
         <transmission name="transmission_${number}">
             <plugin>transmission_interface/SimpleTransmission</plugin>
-            <actuator name="motor_${number}" role="actuator1"/>
-            <joint name="joint_${number}"    role="joint1">
+            <actuator name="motor_${number}" role="actuator1" />
+            <joint name="joint_${number}" role="joint1">
                 <mechanical_reduction>1.0</mechanical_reduction>
             </joint>
@@ -29,134 +31,150 @@
     </xacro:macro>
     <!-- Links -->
-    <link name="world"/>
+    <link name="world" />
     <link name="base_link">
-        <xacro:default_inertial mass="1.0"/>
-        <visual>
-            <origin rpy="0 0 0" xyz="0 0 0.01"/>
-            <geometry>
-                <mesh filename="package://armbot_description/meshes/base_cylinder.stl" scale="0.0001 0.0001 0.0001"/>
+        <xacro:default_inertial mass="1.0" />
+        <visual>
+            <origin rpy="0 0 0" xyz="0 0 0.01" />
+            <geometry>
+                <mesh filename="package://armbot_description/meshes/base_cylinder.stl"
+                    scale="0.0001 0.0001 0.0001" />
             </geometry>
             <material name="black">
-                <color rgba="0 0 0 1"/>
+                <color rgba="0 0 0 1" />
             </material>
         </visual>
         <collision>
-            <origin rpy="0 0 0" xyz="0 0 0.01"/>
-            <geometry>
-                <mesh filename="package://armbot_description/meshes/base_cylinder.stl" scale="0.0001 0.0001 0.0001"/>
+            <origin rpy="0 0 0" xyz="0 0 0.01" />
+            <geometry>
+                <mesh filename="package://armbot_description/meshes/base_cylinder.stl"
+                    scale="0.0001 0.0001 0.0001" />
             </geometry>
         </collision>
     </link>
     <link name="platform">
-        <xacro:default_inertial mass="0.5"/>
-        <visual>
-            <origin rpy="0 0 0" xyz="0 0 0"/>
-            <geometry>
-                <mesh filename="package://armbot_description/meshes/top_plate.stl" scale="0.001 0.001 0.001"/>
-            </geometry>
-            <material name="black"/>
-        </visual>
-        <collision>
-            <origin rpy="0 0 0" xyz="0 0 0"/>
-            <geometry>
-                <mesh filename="package://armbot_description/meshes/top_plate.stl" scale="0.001 0.001 0.001"/>
+        <xacro:default_inertial mass="0.5" />
+        <visual>
+            <origin rpy="0 0 0" xyz="0 0 0" />
+            <geometry>
+                <mesh filename="package://armbot_description/meshes/top_plate.stl"
+                    scale="0.001 0.001 0.001" />
+            </geometry>
+            <material name="black" />
+        </visual>
+        <collision>
+            <origin rpy="0 0 0" xyz="0 0 0" />
+            <geometry>
+                <mesh filename="package://armbot_description/meshes/top_plate.stl"
+                    scale="0.001 0.001 0.001" />
             </geometry>
         </collision>
     </link>
     <link name="lower_arm">
-        <xacro:default_inertial mass="0.5"/>
-        <visual>
-            <origin rpy="0 0 0" xyz="0 0 0"/>
-            <geometry>
-                <mesh filename="package://armbot_description/meshes/lower_arm.stl" scale="0.001 0.001 0.001"/>
-            </geometry>
-            <material name="black"/>
-        </visual>
-        <collision>
-            <origin rpy="0 0 0" xyz="0 0 0"/>
-            <geometry>
-                <mesh filename="package://armbot_description/meshes/lower_arm.stl" scale="0.001 0.001 0.001"/>
+        <xacro:default_inertial mass="0.5" />
+        <visual>
+            <origin rpy="0 0 0" xyz="0 0 0" />
+            <geometry>
+                <mesh filename="package://armbot_description/meshes/lower_arm.stl"
+                    scale="0.001 0.001 0.001" />
+            </geometry>
+            <material name="black" />
+        </visual>
+        <collision>
+            <origin rpy="0 0 0" xyz="0 0 0" />
+            <geometry>
+                <mesh filename="package://armbot_description/meshes/lower_arm.stl"
+                    scale="0.001 0.001 0.001" />
             </geometry>
         </collision>
     </link>
     <link name="top_arm">
-        <xacro:default_inertial mass="0.5"/>
-        <visual>
-            <origin rpy="0 1.59 0" xyz="0 0 0"/>
-            <geometry>
-                <mesh filename="package://armbot_description/meshes/top_arm.stl" scale="0.001 0.001 0.001"/>
-            </geometry>
-            <material name="black"/>
-        </visual>
-        <collision>
-            <origin rpy="0 1.59 0" xyz="0 0 0"/>
-            <geometry>
-                <mesh filename="package://armbot_description/meshes/top_arm.stl" scale="0.001 0.001 0.001"/>
+        <xacro:default_inertial mass="0.5" />
+        <visual>
+            <origin rpy="0 1.59 0" xyz="0 0 0" />
+            <geometry>
+                <mesh filename="package://armbot_description/meshes/top_arm.stl"
+                    scale="0.001 0.001 0.001" />
+            </geometry>
+            <material name="black" />
+        </visual>
+        <collision>
+            <origin rpy="0 1.59 0" xyz="0 0 0" />
+            <geometry>
+                <mesh filename="package://armbot_description/meshes/top_arm.stl"
+                    scale="0.001 0.001 0.001" />
             </geometry>
         </collision>
     </link>
     <link name="wrist">
-        <xacro:default_inertial mass="0.5"/>
-        <visual>
-            <origin rpy="0 0 0" xyz="0 0 0"/>
-            <geometry>
-                <mesh filename="package://armbot_description/meshes/wrist.stl" scale="0.001 0.001 0.001"/>
-            </geometry>
-            <material name="black"/>
-        </visual>
-        <collision>
-            <origin rpy="0 0 0" xyz="0 0 0"/>
-            <geometry>
-                <mesh filename="package://armbot_description/meshes/wrist.stl" scale="0.001 0.001 0.001"/>
+        <xacro:default_inertial mass="0.5" />
+        <visual>
+            <origin rpy="0 0 0" xyz="0 0 0" />
+            <geometry>
+                <mesh filename="package://armbot_description/meshes/wrist.stl"
+                    scale="0.001 0.001 0.001" />
+            </geometry>
+            <material name="black" />
+        </visual>
+        <collision>
+            <origin rpy="0 0 0" xyz="0 0 0" />
+            <geometry>
+                <mesh filename="package://armbot_description/meshes/wrist.stl"
+                    scale="0.001 0.001 0.001" />
             </geometry>
         </collision>
     </link>
     <link name="clawbase">
-        <xacro:default_inertial mass="0.2"/>
-        <visual>
-            <origin rpy="0 3.18 0" xyz="0 0 0"/>
-            <geometry>
-                <mesh filename="package://armbot_description/meshes/clawbase.stl" scale="0.001 0.001 0.001"/>
+        <xacro:default_inertial mass="0.2" />
+        <visual>
+            <origin rpy="0 3.18 0" xyz="0 0 0" />
+            <geometry>
+                <mesh filename="package://armbot_description/meshes/clawbase.stl"
+                    scale="0.001 0.001 0.001" />
             </geometry>
             <material name="white">
-                <color rgba="1 1 1 1"/>
+                <color rgba="1 1 1 1" />
             </material>
         </visual>
         <collision>
-            <origin rpy="0 3.18 0" xyz="0 0 0"/>
-            <geometry>
-                <mesh filename="package://armbot_description/meshes/clawbase.stl" scale="0.001 0.001 0.001"/>
+            <origin rpy="0 3.18 0" xyz="0 0 0" />
+            <geometry>
+                <mesh filename="package://armbot_description/meshes/clawbase.stl"
+                    scale="0.001 0.001 0.001" />
             </geometry>
         </collision>
     </link>
     <link name="clawr">
-        <xacro:default_inertial mass="0.1"/>
-        <visual>
-            <origin rpy="0 0 0" xyz="0 0 0"/>
-            <geometry>
-                <mesh filename="package://armbot_description/meshes/clawr.stl" scale="0.001 0.001 0.001"/>
-            </geometry>
-            <material name="white"/>
-        </visual>
-        <collision>
-            <origin rpy="0 0 0" xyz="0 0 0"/>
-            <geometry>
-                <mesh filename="package://armbot_description/meshes/clawr.stl" scale="0.001 0.001 0.001"/>
+        <xacro:default_inertial mass="0.1" />
+        <visual>
+            <origin rpy="0 0 0" xyz="0 0 0" />
+            <geometry>
+                <mesh filename="package://armbot_description/meshes/clawr.stl"
+                    scale="0.001 0.001 0.001" />
+            </geometry>
+            <material name="white" />
+        </visual>
+        <collision>
+            <origin rpy="0 0 0" xyz="0 0 0" />
+            <geometry>
+                <mesh filename="package://armbot_description/meshes/clawr.stl"
+                    scale="0.001 0.001 0.001" />
             </geometry>
         </collision>
     </link>
     <link name="clawl">
-        <xacro:default_inertial mass="0.1"/>
-        <visual>
-            <origin rpy="0 0 0" xyz="0 0 0"/>
-            <geometry>
-                <mesh filename="package://armbot_description/meshes/clawl.stl" scale="0.001 0.001 0.001"/>
-            </geometry>
-            <material name="white"/>
-        </visual>
-        <collision>
-            <origin rpy="0 0 0" xyz="0 0 0"/>
-            <geometry>
-                <mesh filename="package://armbot_description/meshes/clawl.stl" scale="0.001 0.001 0.001"/>
+        <xacro:default_inertial mass="0.1" />
+        <visual>
+            <origin rpy="0 0 0" xyz="0 0 0" />
+            <geometry>
+                <mesh filename="package://armbot_description/meshes/clawl.stl"
+                    scale="0.001 0.001 0.001" />
+            </geometry>
+            <material name="white" />
+        </visual>
+        <collision>
+            <origin rpy="0 0 0" xyz="0 0 0" />
+            <geometry>
+                <mesh filename="package://armbot_description/meshes/clawl.stl"
+                    scale="0.001 0.001 0.001" />
             </geometry>
         </collision>
@@ -164,57 +182,57 @@
     <!-- Joints -->
     <joint name="virtual_joint" type="fixed">
-        <parent link="world"/>
-        <child link="base_link"/>
-        <origin xyz="0 0 0" rpy="0 0 0"/>
+        <parent link="world" />
+        <child link="base_link" />
+        <origin xyz="0 0 0" rpy="0 0 0" />
     </joint>
     <joint name="joint_1" type="revolute">
         <axis xyz="0 0 1" />
         <limit effort="${effort}" lower="1.56" upper="4.68" velocity="${velocity}" />
-        <parent link="base_link"/>
-        <child link="platform"/>
-        <origin rpy="0 0 1.5" xyz="0 0 0.48"/>
+        <parent link="base_link" />
+        <child link="platform" />
+        <origin rpy="0 0 1.5" xyz="0 0 0.48" />
     </joint>
     <joint name="joint_2" type="revolute">
         <axis xyz="1 0 0" />
         <limit effort="${effort}" lower="0.0" upper="3.12" velocity="${velocity}" />
-        <parent link="platform"/>
-        <child link="lower_arm"/>
-        <origin xyz="0 0.19 0.28"/>
+        <parent link="platform" />
+        <child link="lower_arm" />
+        <origin xyz="0 0.19 0.28" />
     </joint>
     <joint name="joint_3" type="revolute">
         <axis xyz="1 0 0" />
         <limit effort="${effort}" lower="-1.7" upper="1.7" velocity="${velocity}" />
-        <parent link="lower_arm"/>
-        <child link="top_arm"/>
-        <origin xyz="-0.25 1.0 0"/>
+        <parent link="lower_arm" />
+        <child link="top_arm" />
+        <origin xyz="-0.25 1.0 0" />
     </joint>
     <joint name="joint_4" type="revolute">
         <axis xyz="1 0 0" />
         <limit effort="${effort}" lower="-1.7" upper="1.7" velocity="${velocity}" />
-        <parent link="top_arm"/>
-        <child link="wrist"/>
-        <origin xyz="0.11 1.25 0"/>
+        <parent link="top_arm" />
+        <child link="wrist" />
+        <origin xyz="0.11 1.25 0" />
     </joint>
     <joint name="joint_5" type="revolute">
         <axis xyz="0 1 0" />
         <limit effort="${effort}" lower="-3.17" upper="0.0" velocity="${velocity}" />
-        <parent link="wrist"/>
-        <child link="clawbase"/>
-        <origin xyz="0 0.63 0"/>
+        <parent link="wrist" />
+        <child link="clawbase" />
+        <origin xyz="0 0.63 0" />
     </joint>
     <joint name="joint_6" type="revolute">
         <axis xyz="0 0 1" />
         <limit effort="${effort}" lower="-0.5" upper="0.0" velocity="${velocity}" />
-        <parent link="clawbase"/>
-        <child link="clawr"/>
-        <origin rpy="0 0 -0.31" xyz="0.11 0.34 0"/>
+        <parent link="clawbase" />
+        <child link="clawr" />
+        <origin rpy="0 0 -0.31" xyz="0.11 0.34 0" />
     </joint>
     <joint name="joint_7" type="revolute">
         <axis xyz="0 0 1" />
         <limit effort="${effort}" lower="0" upper="-0.5" velocity="${velocity}" />
-        <parent link="clawbase"/>
-        <child link="clawl"/>
-        <origin rpy="0 0 0.22" xyz="-0.16 0.30 0"/>
-        <mimic joint="joint6" multiplier="-1" offset="0" />
+        <parent link="clawbase" />
+        <child link="clawl" />
+        <origin rpy="0 0 0.22" xyz="-0.16 0.30 0" />
+        <mimic joint="joint_6" multiplier="-1" offset="0" />
     </joint>
     <!-- Transmissions -->

File: src/armbot_description/urdf/armbot_gazebo.xacro (robot description, xacro)
@@ -9,3 +9,35 @@
       </plugin>
     </gazebo>
+    <gazebo reference="rgb_camera">
+        <sensor type="camera" name="rgb_camera">
+            <always_on>true</always_on>
+            <update_rate>30.0</update_rate>
+            <camera name="rgb_camera">
+                <horizontal_fov>1.15</horizontal_fov>
+                <vertical_fov>0.71</vertical_fov>
+                <image>
+                    <width>2304</width>
+                    <height>1296</height>
+                    <format>R8G8B8</format>
+                </image>
+                <distortion>
+                    <k1>0.0</k1>
+                    <k2>0.0</k2>
+                    <k3>0.0</k3>
+                    <p1>0.0</p1>
+                    <p2>0.0</p2>
+                    <center>0.5 0.5</center>
+                </distortion>
+            </camera>
+            <plugin name="plugin_name" filename="libgazebo_ros_camera.so">
+                <ros>
+                    <remapping>~/image_raw:=image_raw</remapping>
+                    <remapping>~/camera_info:=camera_info</remapping>
+                </ros>
+                <camera_name>rgb_camera</camera_name>
+                <frame_name>rgb_camera</frame_name>
+                <hack_baseline>0.2</hack_baseline>
+            </plugin>
+        </sensor>
+      </gazebo>
 </robot>

File: src/armbot_description/urdf/armbot_ros2_control.xacro (robot description, xacro)
@@ -4,7 +4,25 @@
         <xacro:property name="PI" value="3.14159265359" />
         <!-- ros2_control Gazebo -->
-        <hardware>
-            <plugin>gazebo_ros2_control/GazeboSystem</plugin>
-        </hardware>
+        <xacro:if value="$(arg is_sim)">
+            <hardware>
+                <plugin>gazebo_ros2_control/GazeboSystem</plugin>
+            </hardware>
+            <joint name="joint_7">
+                <param name="mimic">joint_6</param>
+                <param name="multiplier">-1</param>
+                <command_interface name="position">
+                <param name="min">0.0</param>
+                <param name="max">${PI / 2}</param>
+                </command_interface>
+            </joint>
+        </xacro:if>
+        <!-- ros2_control Real Robot -->
+        <xacro:unless value="$(arg is_sim)">
+            <hardware>
+                <plugin>armbot_controller/ArmbotInterface</plugin>
+                <param name="port">/dev/ttyACM0</param>
+            </hardware>
+        </xacro:unless>
+        <!-- ros2_control Common Interfaces -->
         <joint name="joint_1">
             <command_interface name="position">
@@ -12,5 +30,5 @@
                 <param name="max">${PI / 2}</param>
             </command_interface>
-            <state_interface name="position"/>
+            <state_interface name="position" />
         </joint>
         <joint name="joint_2">
@@ -19,5 +37,5 @@
                 <param name="max">${PI / 2}</param>
             </command_interface>
-            <state_interface name="position"/>
+            <state_interface name="position" />
         </joint>
         <joint name="joint_3">
@@ -26,5 +44,5 @@
                 <param name="max">${PI / 2}</param>
             </command_interface>
-            <state_interface name="position"/>
+            <state_interface name="position" />
         </joint>
         <joint name="joint_4">
@@ -33,5 +51,5 @@
                 <param name="max">${PI / 2}</param>
             </command_interface>
-            <state_interface name="position"/>
+            <state_interface name="position" />
         </joint>
         <joint name="joint_5">
@@ -40,7 +58,6 @@
                 <param name="max">${PI / 2}</param>
             </command_interface>
-            <state_interface name="position"/>
+            <state_interface name="position" />
         </joint>
-        <!-- New joints for 6-DOF -->
         <joint name="joint_6">
             <command_interface name="position">
@@ -48,13 +65,5 @@
                 <param name="max">0.0</param>
             </command_interface>
-            <state_interface name="position"/>
-        </joint>
-        <joint name="joint_7">
-            <param name="mimic">joint_6</param>
-            <param name="multiplier">-1</param>
-            <command_interface name="position">
-                <param name="min">0.0</param>
-                <param name="max">${PI / 2}</param>
-            </command_interface>
+            <state_interface name="position" />
         </joint>
     </ros2_control>
