Commit message: description migrate to jazzy

File: src/armbot_description/urdf/armbot.urdf.xacro (robot description, xacro)
@@ -37,6 +37,5 @@
             <origin rpy="0 0 0" xyz="0 0 0.01" />
             <geometry>
-                <mesh filename="package://armbot_description/meshes/base_cylinder.stl"
-                    scale="0.0001 0.0001 0.0001" />
+                <mesh filename="package://armbot_description/meshes/base_cylinder.stl" scale="0.0001 0.0001 0.0001" />
             </geometry>
             <material name="black">
@@ -47,6 +46,5 @@
             <origin rpy="0 0 0" xyz="0 0 0.01" />
             <geometry>
-                <mesh filename="package://armbot_description/meshes/base_cylinder.stl"
-                    scale="0.0001 0.0001 0.0001" />
+                <mesh filename="package://armbot_description/meshes/base_cylinder.stl" scale="0.0001 0.0001 0.0001" />
             </geometry>
         </collision>
@@ -57,14 +55,12 @@
             <origin rpy="0 0 0" xyz="0 0 0" />
             <geometry>
-                <mesh filename="package://armbot_description/meshes/top_plate.stl"
-                    scale="0.001 0.001 0.001" />
-            </geometry>
-            <material name="black" />
-        </visual>
-        <collision>
-            <origin rpy="0 0 0" xyz="0 0 0" />
-            <geometry>
-                <mesh filename="package://armbot_description/meshes/top_plate.stl"
-                    scale="0.001 0.001 0.001" />
+                <mesh filename="package://armbot_description/meshes/top_plate.stl" scale="0.001 0.001 0.001" />
+            </geometry>
+            <material name="black" />
+        </visual>
+        <collision>
+            <origin rpy="0 0 0" xyz="0 0 0" />
+            <geometry>
+                <mesh filename="package://armbot_description/meshes/top_plate.stl" scale="0.001 0.001 0.001" />
             </geometry>
         </collision>
@@ -75,14 +71,12 @@
             <origin rpy="0 0 0" xyz="0 0 0" />
             <geometry>
-                <mesh filename="package://armbot_description/meshes/lower_arm.stl"
-                    scale="0.001 0.001 0.001" />
-            </geometry>
-            <material name="black" />
-        </visual>
-        <collision>
-            <origin rpy="0 0 0" xyz="0 0 0" />
-            <geometry>
-                <mesh filename="package://armbot_description/meshes/lower_arm.stl"
-                    scale="0.001 0.001 0.001" />
+                <mesh filename="package://armbot_description/meshes/lower_arm.stl" scale="0.001 0.001 0.001" />
+            </geometry>
+            <material name="black" />
+        </visual>
+        <collision>
+            <origin rpy="0 0 0" xyz="0 0 0" />
+            <geometry>
+                <mesh filename="package://armbot_description/meshes/lower_arm.stl" scale="0.001 0.001 0.001" />
             </geometry>
         </collision>
@@ -93,6 +87,5 @@
             <origin rpy="0 1.59 0" xyz="0 0 0" />
             <geometry>
-                <mesh filename="package://armbot_description/meshes/top_arm.stl"
-                    scale="0.001 0.001 0.001" />
+                <mesh filename="package://armbot_description/meshes/top_arm.stl" scale="0.001 0.001 0.001" />
             </geometry>
             <material name="black" />
@@ -101,6 +94,5 @@
             <origin rpy="0 1.59 0" xyz="0 0 0" />
             <geometry>
-                <mesh filename="package://armbot_description/meshes/top_arm.stl"
-                    scale="0.001 0.001 0.001" />
+                <mesh filename="package://armbot_description/meshes/top_arm.stl" scale="0.001 0.001 0.001" />
             </geometry>
         </collision>
@@ -111,14 +103,12 @@
             <origin rpy="0 0 0" xyz="0 0 0" />
             <geometry>
-                <mesh filename="package://armbot_description/meshes/wrist.stl"
-                    scale="0.001 0.001 0.001" />
-            </geometry>
-            <material name="black" />
-        </visual>
-        <collision>
-            <origin rpy="0 0 0" xyz="0 0 0" />
-            <geometry>
-                <mesh filename="package://armbot_description/meshes/wrist.stl"
-                    scale="0.001 0.001 0.001" />
+                <mesh filename="package://armbot_description/meshes/wrist.stl" scale="0.001 0.001 0.001" />
+            </geometry>
+            <material name="black" />
+        </visual>
+        <collision>
+            <origin rpy="0 0 0" xyz="0 0 0" />
+            <geometry>
+                <mesh filename="package://armbot_description/meshes/wrist.stl" scale="0.001 0.001 0.001" />
             </geometry>
         </collision>
@@ -129,6 +119,5 @@
             <origin rpy="0 3.18 0" xyz="0 0 0" />
             <geometry>
-                <mesh filename="package://armbot_description/meshes/clawbase.stl"
-                    scale="0.001 0.001 0.001" />
+                <mesh filename="package://armbot_description/meshes/clawbase.stl" scale="0.001 0.001 0.001" />
             </geometry>
             <material name="white">
@@ -139,6 +128,5 @@
             <origin rpy="0 3.18 0" xyz="0 0 0" />
             <geometry>
-                <mesh filename="package://armbot_description/meshes/clawbase.stl"
-                    scale="0.001 0.001 0.001" />
+                <mesh filename="package://armbot_description/meshes/clawbase.stl" scale="0.001 0.001 0.001" />
             </geometry>
         </collision>
@@ -149,6 +137,5 @@
             <origin rpy="0 0 0" xyz="0 0 0" />
             <geometry>
-                <mesh filename="package://armbot_description/meshes/clawr.stl"
-                    scale="0.001 0.001 0.001" />
+                <mesh filename="package://armbot_description/meshes/clawr.stl" scale="0.001 0.001 0.001" />
             </geometry>
             <material name="white" />
@@ -157,6 +144,5 @@
             <origin rpy="0 0 0" xyz="0 0 0" />
             <geometry>
-                <mesh filename="package://armbot_description/meshes/clawr.stl"
-                    scale="0.001 0.001 0.001" />
+                <mesh filename="package://armbot_description/meshes/clawr.stl" scale="0.001 0.001 0.001" />
             </geometry>
         </collision>
@@ -167,6 +153,5 @@
             <origin rpy="0 0 0" xyz="0 0 0" />
             <geometry>
-                <mesh filename="package://armbot_description/meshes/clawl.stl"
-                    scale="0.001 0.001 0.001" />
+                <mesh filename="package://armbot_description/meshes/clawl.stl" scale="0.001 0.001 0.001" />
             </geometry>
             <material name="white" />
@@ -175,6 +160,23 @@
             <origin rpy="0 0 0" xyz="0 0 0" />
             <geometry>
-                <mesh filename="package://armbot_description/meshes/clawl.stl"
-                    scale="0.001 0.001 0.001" />
+                <mesh filename="package://armbot_description/meshes/clawl.stl" scale="0.001 0.001 0.001" />
+            </geometry>
+        </collision>
+    </link>
+    <link name="camera">
+        <xacro:default_inertial mass="0.05" />
+        <visual>
+            <origin rpy="-1.57 0 -1.57" xyz="0.1 0.2 0.15" />
+            <geometry>
+                <mesh filename="package://armbot_description/meshes/pi_camera.STL" scale="0.01 0.01 0.01" />
+            </geometry>
+            <material name="gray">
+                <color rgba="0.5 0.5 0.5 1" />
+            </material>
+        </visual>
+        <collision>
+            <origin rpy="-1.57 0 -1.57" xyz="0.1 0.2 0.15" />
+            <geometry>
+                <mesh filename="package://armbot_description/meshes/pi_camera.STL" scale="0.01 0.01 0.01" />
             </geometry>
         </collision>
@@ -235,4 +237,9 @@
         <origin rpy="0 0 0.22" xyz="-0.16 0.30 0" />
         <mimic joint="joint_6" multiplier="-1" offset="0" />
+    </joint>
+    <joint name="camera_joint" type="fixed">
+        <parent link="base_link" />
+        <child link="camera" />
+        <origin xyz="0 0.45 0.2" rpy="0 -0.5 1.57" />
     </joint>
     <!-- Transmissions -->

File: src/armbot_description/urdf/armbot_gazebo.xacro (robot description, xacro)
@@ -1,43 +1,39 @@
 <?xml version="1.0"?>
 <robot xmlns:xacro="http://www.ros.org/wiki/xacro" name="armbot">
-    <!-- Gazebo ros2_control plugin -->
-    <gazebo>
-        <plugin name="gz_ros2_control::GazeboSimROS2ControlPlugin" filename="libgz_ros2_control-system.so">
-        <robot_param>robot_description</robot_param>
-        <robot_param_node>robot_state_publisher</robot_param_node>
-        <parameters>$(find armbot_controller)/config/armbot_controllers.yaml</parameters>
-      </plugin>
-    </gazebo>
-    <gazebo reference="rgb_camera">
-        <sensor type="camera" name="rgb_camera">
-            <always_on>true</always_on>
-            <update_rate>30.0</update_rate>
-            <camera name="rgb_camera">
-                <horizontal_fov>1.15</horizontal_fov>
-                <vertical_fov>0.71</vertical_fov>
-                <image>
-                    <width>2304</width>
-                    <height>1296</height>
-                    <format>R8G8B8</format>
-                </image>
-                <distortion>
-                    <k1>0.0</k1>
-                    <k2>0.0</k2>
-                    <k3>0.0</k3>
-                    <p1>0.0</p1>
-                    <p2>0.0</p2>
-                    <center>0.5 0.5</center>
-                </distortion>
-            </camera>
-            <plugin name="plugin_name" filename="libgazebo_ros_camera.so">
-                <ros>
-                    <remapping>~/image_raw:=image_raw</remapping>
-                    <remapping>~/camera_info:=camera_info</remapping>
-                </ros>
-                <camera_name>rgb_camera</camera_name>
-                <frame_name>rgb_camera</frame_name>
-                <hack_baseline>0.2</hack_baseline>
-            </plugin>
-        </sensor>
-      </gazebo>
+  <!-- ROS 2 Control -->
+  <gazebo>
+    <!-- ROS 2 Iron or Jazzy or above -->
+    <plugin filename="gz_ros2_control-system" name="gz_ros2_control::GazeboSimROS2ControlPlugin">
+      <parameters>$(find armbot_controller)/config/armbot_controllers.yaml</parameters>
+    </plugin>
+    <plugin filename="gz-sim-sensors-system" name="gz::sim::systems::Sensors">
+      <render_engine>ogre2</render_engine>
+    </plugin>
+  </gazebo>
+  <!-- Camera sensor setup -->
+  <gazebo reference="camera">
+    <sensor name="camera" type="camera">
+      <always_on>true</always_on>
+      <update_rate>30.0</update_rate>
+      <visualize>true</visualize>
+      <topic>/image_raw</topic>
+      <gz_frame_id>/camera</gz_frame_id>
+      <camera name="camera">
+        <horizontal_fov>1.21126</horizontal_fov>
+        <image>
+          <width>2304</width>
+          <height>1296</height>
+          <format>R8G8B8</format>
+        </image>
+        <distortion>
+          <k1>0.0</k1>
+          <k2>0.0</k2>
+          <k3>0.0</k3>
+          <p1>0.0</p1>
+          <p2>0.0</p2>
+          <center>0.5 0.5</center>
+        </distortion>
+      </camera>
+    </sensor>
+  </gazebo>
 </robot>

File: src/armbot_description/urdf/armbot_ros2_control.xacro (robot description, xacro)
@@ -5,19 +5,8 @@
         <!-- ros2_control Gazebo -->
         <xacro:if value="$(arg is_sim)">
+            <!-- GazeboSimSystem for ROS 2 Jazzy -->
             <hardware>
                 <plugin>gz_ros2_control/GazeboSimSystem</plugin>
             </hardware>
-            <hardware>
-                <plugin>armbot_controller/ArmbotInterface</plugin>
-                <param name="port">/dev/ttyACM0</param>
-            </hardware>
-            <joint name="joint_7">
-                <param name="mimic">joint_6</param>
-                <param name="multiplier">-1</param>
-                <command_interface name="position">
-                <param name="min">0.0</param>
-                <param name="max">${PI / 2}</param>
-                </command_interface>
-            </joint>
         </xacro:if>
         <!-- ros2_control Real Robot -->
@@ -71,4 +60,9 @@
             <state_interface name="position" />
         </joint>
+        <!-- Mimic joint configuration -->
+        <joint name="joint_7">
+            <param name="mimic">joint_6</param>
+            <param name="multiplier">-1</param>
+        </joint>
     </ros2_control>
 </robot>
