Commit message: re-factor

File: src/armbot_description/urdf/armbot.urdf.xacro (robot description, xacro)
@@ -37,5 +37,6 @@
             <origin rpy="0 0 0" xyz="0 0 0.01" />
             <geometry>
-                <mesh filename="package://armbot_description/meshes/base_cylinder.stl" scale="0.0001 0.0001 0.0001" />
+                <mesh filename="package://armbot_description/meshes/base_cylinder.stl"
+                    scale="0.0001 0.0001 0.0001" />
             </geometry>
             <material name="black">
@@ -46,5 +47,6 @@
             <origin rpy="0 0 0" xyz="0 0 0.01" />
             <geometry>
-                <mesh filename="package://armbot_description/meshes/base_cylinder.stl" scale="0.0001 0.0001 0.0001" />
+                <mesh filename="package://armbot_description/meshes/base_cylinder.stl"
+                    scale="0.0001 0.0001 0.0001" />
             </geometry>
         </collision>
@@ -55,12 +57,14 @@
             <origin rpy="0 0 0" xyz="0 0 0" />
             <geometry>
-                <mesh filename="package://armbot_description/meshes/top_plate.stl" scale="0.001 0.001 0.001" />
-            </geometry>
-            <material name="black" />
-        </visual>
-        <collision>
-            <origin rpy="0 0 0" xyz="0 0 0" />
-            <geometry>
-                <mesh filename="package://armbot_description/meshes/top_plate.stl" scale="0.001 0.001 0.001" />
+                <mesh filename="package://armbot_description/meshes/top_plate.stl"
+                    scale="0.001 0.001 0.001" />
+            </geometry>
+            <material name="black" />
+        </visual>
+        <collision>
+            <origin rpy="0 0 0" xyz="0 0 0" />
+            <geometry>
+                <mesh filename="package://armbot_description/meshes/top_plate.stl"
+                    scale="0.001 0.001 0.001" />
             </geometry>
         </collision>
@@ -71,12 +75,14 @@
             <origin rpy="0 0 0" xyz="0 0 0" />
             <geometry>
-                <mesh filename="package://armbot_description/meshes/lower_arm.stl" scale="0.001 0.001 0.001" />
-            </geometry>
-            <material name="black" />
-        </visual>
-        <collision>
-            <origin rpy="0 0 0" xyz="0 0 0" />
-            <geometry>
-                <mesh filename="package://armbot_description/meshes/lower_arm.stl" scale="0.001 0.001 0.001" />
+                <mesh filename="package://armbot_description/meshes/lower_arm.stl"
+                    scale="0.001 0.001 0.001" />
+            </geometry>
+            <material name="black" />
+        </visual>
+        <collision>
+            <origin rpy="0 0 0" xyz="0 0 0" />
+            <geometry>
+                <mesh filename="package://armbot_description/meshes/lower_arm.stl"
+                    scale="0.001 0.001 0.001" />
             </geometry>
         </collision>
@@ -87,5 +93,6 @@
             <origin rpy="0 1.59 0" xyz="0 0 0" />
             <geometry>
-                <mesh filename="package://armbot_description/meshes/top_arm.stl" scale="0.001 0.001 0.001" />
+                <mesh filename="package://armbot_description/meshes/top_arm.stl"
+                    scale="0.001 0.001 0.001" />
             </geometry>
             <material name="black" />
@@ -94,5 +101,6 @@
             <origin rpy="0 1.59 0" xyz="0 0 0" />
             <geometry>
-                <mesh filename="package://armbot_description/meshes/top_arm.stl" scale="0.001 0.001 0.001" />
+                <mesh filename="package://armbot_description/meshes/top_arm.stl"
+                    scale="0.001 0.001 0.001" />
             </geometry>
         </collision>
@@ -103,12 +111,14 @@
             <origin rpy="0 0 0" xyz="0 0 0" />
             <geometry>
-                <mesh filename="package://armbot_description/meshes/wrist.stl" scale="0.001 0.001 0.001" />
-            </geometry>
-            <material name="black" />
-        </visual>
-        <collision>
-            <origin rpy="0 0 0" xyz="0 0 0" />
-            <geometry>
-                <mesh filename="package://armbot_description/meshes/wrist.stl" scale="0.001 0.001 0.001" />
+                <mesh filename="package://armbot_description/meshes/wrist.stl"
+                    scale="0.001 0.001 0.001" />
+            </geometry>
+            <material name="black" />
+        </visual>
+        <collision>
+            <origin rpy="0 0 0" xyz="0 0 0" />
+            <geometry>
+                <mesh filename="package://armbot_description/meshes/wrist.stl"
+                    scale="0.001 0.001 0.001" />
             </geometry>
         </collision>
@@ -119,5 +129,6 @@
             <origin rpy="0 3.18 0" xyz="0 0 0" />
             <geometry>
-                <mesh filename="package://armbot_description/meshes/clawbase.stl" scale="0.001 0.001 0.001" />
+                <mesh filename="package://armbot_description/meshes/clawbase.stl"
+                    scale="0.001 0.001 0.001" />
             </geometry>
             <material name="white">
@@ -128,5 +139,6 @@
             <origin rpy="0 3.18 0" xyz="0 0 0" />
             <geometry>
-                <mesh filename="package://armbot_description/meshes/clawbase.stl" scale="0.001 0.001 0.001" />
+                <mesh filename="package://armbot_description/meshes/clawbase.stl"
+                    scale="0.001 0.001 0.001" />
             </geometry>
         </collision>
@@ -137,5 +149,6 @@
             <origin rpy="0 0 0" xyz="0 0 0" />
             <geometry>
-                <mesh filename="package://armbot_description/meshes/clawr.stl" scale="0.001 0.001 0.001" />
+                <mesh filename="package://armbot_description/meshes/clawr.stl"
+                    scale="0.001 0.001 0.001" />
             </geometry>
             <material name="white" />
@@ -144,5 +157,6 @@
             <origin rpy="0 0 0" xyz="0 0 0" />
             <geometry>
-                <mesh filename="package://armbot_description/meshes/clawr.stl" scale="0.001 0.001 0.001" />
+                <mesh filename="package://armbot_description/meshes/clawr.stl"
+                    scale="0.001 0.001 0.001" />
             </geometry>
         </collision>
@@ -153,5 +167,6 @@
             <origin rpy="0 0 0" xyz="0 0 0" />
             <geometry>
-                <mesh filename="package://armbot_description/meshes/clawl.stl" scale="0.001 0.001 0.001" />
+                <mesh filename="package://armbot_description/meshes/clawl.stl"
+                    scale="0.001 0.001 0.001" />
             </geometry>
             <material name="white" />
@@ -160,23 +175,6 @@
             <origin rpy="0 0 0" xyz="0 0 0" />
             <geometry>
-                <mesh filename="package://armbot_description/meshes/clawl.stl" scale="0.001 0.001 0.001" />
-            </geometry>
-        </collision>
-    </link>
-    <link name="camera">
-        <xacro:default_inertial mass="0.05" />
-        <visual>
-            <origin rpy="-1.57 0 -1.57" xyz="0.1 0.2 0.15" />
-            <geometry>
-                <mesh filename="package://armbot_description/meshes/pi_camera.STL" scale="0.01 0.01 0.01" />
-            </geometry>
-            <material name="gray">
-                <color rgba="0.5 0.5 0.5 1" />
-            </material>
-        </visual>
-        <collision>
-            <origin rpy="-1.57 0 -1.57" xyz="0.1 0.2 0.15" />
-            <geometry>
-                <mesh filename="package://armbot_description/meshes/pi_camera.STL" scale="0.01 0.01 0.01" />
+                <mesh filename="package://armbot_description/meshes/clawl.stl"
+                    scale="0.001 0.001 0.001" />
             </geometry>
         </collision>
@@ -237,9 +235,4 @@
         <origin rpy="0 0 0.22" xyz="-0.16 0.30 0" />
         <mimic joint="joint_6" multiplier="-1" offset="0" />
-    </joint>
-    <joint name="camera_joint" type="fixed">
-        <parent link="base_link" />
-        <child link="camera" />
-        <origin xyz="0 0.45 0.2" rpy="0 -0.5 1.57" />
     </joint>
     <!-- Transmissions -->

File: src/armbot_description/urdf/armbot_gazebo.xacro (robot description, xacro)
@@ -1,39 +1,38 @@
 <?xml version="1.0"?>
 <robot xmlns:xacro="http://www.ros.org/wiki/xacro" name="armbot">
-  <!-- ROS 2 Control -->
-  <gazebo>
-    <!-- ROS 2 Iron or Jazzy or above -->
-    <plugin filename="gz_ros2_control-system" name="gz_ros2_control::GazeboSimROS2ControlPlugin">
-      <parameters>$(find armbot_controller)/config/armbot_controllers.yaml</parameters>
-    </plugin>
-    <plugin filename="gz-sim-sensors-system" name="gz::sim::systems::Sensors">
-      <render_engine>ogre2</render_engine>
-    </plugin>
-  </gazebo>
-  <!-- Camera sensor setup -->
-  <gazebo reference="camera">
-    <sensor name="camera" type="camera">
-      <always_on>true</always_on>
-      <update_rate>30.0</update_rate>
-      <visualize>true</visualize>
-      <topic>/image_raw</topic>
-      <gz_frame_id>/camera</gz_frame_id>
-      <camera name="camera">
-        <horizontal_fov>1.21126</horizontal_fov>
-        <image>
-          <width>2304</width>
-          <height>1296</height>
-          <format>R8G8B8</format>
-        </image>
-        <distortion>
-          <k1>0.0</k1>
-          <k2>0.0</k2>
-          <k3>0.0</k3>
-          <p1>0.0</p1>
-          <p2>0.0</p2>
-          <center>0.5 0.5</center>
-        </distortion>
-      </camera>
-    </sensor>
-  </gazebo>
+    <!-- Gazebo plugin setup for ROS 2 Jazzy -->
+    <gazebo>
+        <plugin filename="gz_ros2_control-system" name="gz_ros2_control::GazeboSimROS2ControlPlugin">
+            <parameters>$(find armbot_controller)/config/armbot_controllers.yaml</parameters>
+        </plugin>
+        <plugin filename="gz-sim-sensors-system" name="gz::sim::systems::Sensors">
+            <render_engine>ogre2</render_engine>
+        </plugin>
+    </gazebo>
+    <!-- Camera sensor configuration -->
+    <gazebo reference="camera">
+        <sensor name="camera" type="camera">
+            <always_on>true</always_on>
+            <update_rate>30.0</update_rate>
+            <visualize>true</visualize>
+            <topic>/image_raw</topic>
+            <gz_frame_id>/camera</gz_frame_id>
+            <camera name="camera">
+                <horizontal_fov>1.21126</horizontal_fov>
+                <image>
+                    <width>2304</width>
+                    <height>1296</height>
+                    <format>R8G8B8</format>
+                </image>
+                <distortion>
+                    <k1>0.0</k1>
+                    <k2>0.0</k2>
+                    <k3>0.0</k3>
+                    <p1>0.0</p1>
+                    <p2>0.0</p2>
+                    <center>0.5 0.5</center>
+                </distortion>
+            </camera>
+        </sensor>
+    </gazebo>
 </robot>

File: src/armbot_description/urdf/armbot_ros2_control.xacro (robot description, xacro)
@@ -1,63 +1,41 @@
 <?xml version="1.0"?>
 <robot xmlns:xacro="http://www.ros.org/wiki/xacro" name="armbot">
+    <!-- ROS 2 Control System -->
     <ros2_control name="RobotSystem" type="system">
+        <!-- Define common properties -->
         <xacro:property name="PI" value="3.14159265359" />
-        <!-- ros2_control Gazebo -->
-        <xacro:if value="$(arg is_sim)">
-            <!-- GazeboSimSystem for ROS 2 Jazzy -->
-            <hardware>
-                <plugin>gz_ros2_control/GazeboSimSystem</plugin>
-            </hardware>
-        </xacro:if>
-        <!-- ros2_control Real Robot -->
-        <xacro:unless value="$(arg is_sim)">
-            <hardware>
-                <plugin>armbot_controller/ArmbotInterface</plugin>
-                <param name="port">/dev/ttyACM0</param>
-            </hardware>
-        </xacro:unless>
-        <!-- ros2_control Common Interfaces -->
-        <joint name="joint_1">
-            <command_interface name="position">
-                <param name="min">-${PI / 2}</param>
-                <param name="max">${PI / 2}</param>
-            </command_interface>
-            <state_interface name="position" />
-        </joint>
-        <joint name="joint_2">
-            <command_interface name="position">
-                <param name="min">-${PI / 2}</param>
-                <param name="max">${PI / 2}</param>
-            </command_interface>
-            <state_interface name="position" />
-        </joint>
-        <joint name="joint_3">
-            <command_interface name="position">
-                <param name="min">-${PI / 2}</param>
-                <param name="max">${PI / 2}</param>
-            </command_interface>
-            <state_interface name="position" />
-        </joint>
-        <joint name="joint_4">
-            <command_interface name="position">
-                <param name="min">-${PI / 2}</param>
-                <param name="max">${PI / 2}</param>
-            </command_interface>
-            <state_interface name="position" />
-        </joint>
-        <joint name="joint_5">
-            <command_interface name="position">
-                <param name="min">-${PI / 2}</param>
-                <param name="max">${PI / 2}</param>
-            </command_interface>
-            <state_interface name="position" />
-        </joint>
-        <joint name="joint_6">
-            <command_interface name="position">
-                <param name="min">-${PI / 2}</param>
-                <param name="max">0.0</param>
-            </command_interface>
-            <state_interface name="position" />
-        </joint>
+        <!-- Hardware interface setup -->
+        <xacro:macro name="hardware_interface" params="is_sim plugin_name port">
+            <xacro:if value="${is_sim}">
+                <hardware>
+                    <plugin>${plugin_name}</plugin>
+                </hardware>
+            </xacro:if>
+            <xacro:unless value="${is_sim}">
+                <hardware>
+                    <plugin>armbot_controller/ArmbotInterface</plugin>
+                    <param name="port">${port}</param>
+                </hardware>
+            </xacro:unless>
+        </xacro:macro>
+        <!-- Invoke hardware interface for simulation or real robot -->
+        <xacro:hardware_interface is_sim="$(arg is_sim)" plugin_name="gz_ros2_control/GazeboSimSystem" port="/dev/ttyACM0" />
+        <!-- Common joint interface macro -->
+        <xacro:macro name="joint_interface" params="joint_name min_angle max_angle">
+            <joint name="${joint_name}">
+                <command_interface name="position">
+                    <param name="min">${min_angle}</param>
+                    <param name="max">${max_angle}</param>
+                </command_interface>
+                <state_interface name="position" />
+            </joint>
+        </xacro:macro>
+        <!-- Define joint interfaces -->
+        <xacro:joint_interface joint_name="joint_1" min_angle="-${PI / 2}" max_angle="${PI / 2}" />
+        <xacro:joint_interface joint_name="joint_2" min_angle="-${PI / 2}" max_angle="${PI / 2}" />
+        <xacro:joint_interface joint_name="joint_3" min_angle="-${PI / 2}" max_angle="${PI / 2}" />
+        <xacro:joint_interface joint_name="joint_4" min_angle="-${PI / 2}" max_angle="${PI / 2}" />
+        <xacro:joint_interface joint_name="joint_5" min_angle="-${PI / 2}" max_angle="${PI / 2}" />
+        <xacro:joint_interface joint_name="joint_6" min_angle="-${PI / 2}" max_angle="0.0" />
         <!-- Mimic joint configuration -->
         <joint name="joint_7">
